File: kicad/apd.kicad_pcb (KiCad board)
At the start: 2 copper layers, 22 x 21.6 mm, 26 parts, among them IC1 LT3571EUD#PBF, IC2 ATSAMD21E18A-AFT, IC3 ADP7118ACPZN3.3, J1 Conn_01x04, J2 CX80B1-24P, J3 Conn_01x03, U1 MCP4726A0T-E_MAY

Commit message: routed v100
Parts:
- removed D1: LED, footprints:D_0603_1608Metric_Castellated
- removed R7: 1k, footprints:R_0402_1005Metric
- moved C9 55.7 mm to (195.7, 94.1), turned to 270 degrees
- moved C4 53.8 mm to (201.6, 100.1)
- moved C10 47.7 mm to (192.7, 95.5)
- moved C2 47.2 mm to (197.3, 108.8), turned to 90 degrees
- moved R9 45.5 mm to (195.6, 91.8), turned to 180 degrees
- moved R8 43.9 mm to (198.5, 100.7), turned to 180 degrees
- moved C1 43.6 mm to (196.1, 108.8), turned to 90 degrees
- moved C7 42.6 mm to (192.5, 100.3), turned to 90 degrees
- moved R2 42.4 mm to (200.6, 107.1), turned to 180 degrees
- moved IC3 34.1 mm to (193.4, 93.9)
- moved J1 25.4 mm to (190.4, 99.8), turned to 90 degrees
- moved IC2 16.2 mm to (195.6, 104.1), turned to 45 degrees
- moved IC1 0.70 mm to (203.9, 106.0)
- moved L1 0.70 mm to (201.1, 103.2)
- moved U1 0.52 mm to (199.1, 109.1)
Connections:
- net /USB_DM renamed /USB_DN
- IC2 pad 13: Net-(IC2-Pad13) -> /~SHDN
- IC2 pad 33: (no net) -> GND
- IC3 pad 1: +5V -> +3V3
- IC3 pad 2: GND -> +3V3
- IC3 pad 3: +5V -> GND
- IC3 pad 4: +3V3 -> +5V
- IC3 pad 5: +3V3 -> (no net)
- IC3 pad 6: (no net) -> +5V
- IC3 pad 7: (no net) -> GND
Routing:
- net +3V3: track 0.00 -> 36.7 mm, vias 0 -> 1
- net +5V: track 3.40 -> 34.0 mm
- net GND: track 10.3 -> 29.9 mm, vias 9 -> 19
- net /USB_DP: track 0.00 -> 11.9 mm, vias 0 -> 3
- net /USB_DN: track 0.00 -> 8.14 mm
- net Net-(J2-PadA5): track 0.00 -> 6.45 mm
- net /RESET: track 0.00 -> 6.28 mm
- net /~SHDN: track 0.00 -> 6.05 mm
- net Net-(IC1-Pad9): track 0.00 -> 5.18 mm, vias 0 -> 2
- net /SWCLK: track 0.00 -> 5.11 mm
- net /SWDIO: track 0.00 -> 4.12 mm
- net /SCL: track 0.00 -> 3.86 mm
- net Net-(J2-PadB5): track 0.00 -> 3.63 mm
- net /SDA: track 0.00 -> 3.41 mm
- net Net-(C7-Pad1): track 0.00 -> 1.99 mm
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- added copper zone on F.Cu, net (none)
Other:
- board text added: "SiPM Bias"
- board text added: "v100"
