File: kicad/apd.sch (KiCad schematic (older format))
At the start: 26 parts, among them IC1 LT3571EUD#PBF, IC2 ATSAMD21E18A-AFT, IC3 ADP7118ACPZN3.3, J1 Conn_01x04, J2 CX80B1-24P, J3 Conn_01x03, U1 MCP4726A0T-E_MAY

Commit message: routed v100
Parts:
- removed D1: LED, D_0603_1608Metric_Castellated, symbol Device:LED
- removed R7: 1k, R_0402_1005Metric, symbol Device:R_Small_US
Connections:
- net labels added: USB_DN
- net labels removed: USB_DM
- wire segments 134 -> 130
- no-connect marks 11 -> 12
Other:
- moved on the sheet: C10
Changed lines of the file:
@@
 Connection ~ 1425 4850
 Text Label 5975 2425 2    50   ~ 0
-USB_DM
+USB_DN
 Text Label 5975 2525 2    50   ~ 0
 USB_DP
@@
 	8925 3200 9225 3200
 Text Label 8925 3100 0    50   ~ 0
-USB_DM
+USB_DN
 Text Label 8925 3200 0    50   ~ 0
 USB_DP
@@
 Text Label 7275 1300 0    50   ~ 0
 RESET
-$Comp
-L Device:R_Small_US R7
-U 1 1 5BFE5A5C
-P 9775 2450
-F 0 "R7" H 9843 2496 50  0000 L CNN
-F 1 "1k" H 9843 2405 50  0000 L CNN
-F 2 "R_0402_1005Metric" H 9775 2450 50  0001 C CNN
-F 3 "~" H 9775 2450 50  0001 C CNN
-	1    9775 2450
-	1    0    0    -1
-$EndComp
-$Comp
-L Device:LED D1
-U 1 1 5BFE5A63
-P 9775 2900
-F 0 "D1" V 9813 2783 50  0000 R CNN
-F 1 "LED" V 9722 2783 50  0000 R CNN
-F 2 "D_0603_1608Metric_Castellated" H 9775 2900 50  0001 C CNN
-F 3 "~" H 9775 2900 50  0001 C CNN
-	1    9775 2900
-	0    -1   -1   0
-$EndComp
-Wire Wire Line
-	9775 2550 9775 2750
-$Comp
-L power:GND #PWR0115
-U 1 1 5BFE5A6C
-P 9775 3150
-F 0 "#PWR0115" H 9775 2900 50  0001 C CNN
-F 1 "GND" H 9780 2977 50  0000 C CNN
-F 2 "" H 9775 3150 50  0001 C CNN
-F 3 "" H 9775 3150 50  0001 C CNN
-	1    9775 3150
-	1    0    0    -1
-$EndComp
-Wire Wire Line
-	9775 3050 9775 3150
-Wire Wire Line
-	8925 2100 9775 2100
-Wire Wire Line
-	9775 2100 9775 2350
 Text Label 9075 2000 2    50   ~ 0
 SCL
@@
 Wire Wire Line
 	1400 2150 1825 2150
-Wire Wire Line
-	2775 2050 2825 2050
-Wire Wire Line
-	2825 2050 2825 1950
-Wire Wire Line
-	2825 1950 2775 1950
 $Comp
 L Device:C_Small C10
 U 1 1 5DC20B68
-P 2975 1975
-F 0 "C10" H 3067 2021 50  0000 L CNN
-F 1 "2.2u" H 3067 1930 50  0000 L CNN
-F 2 "C_0402_1005Metric" H 2975 1975 50  0001 C CNN
-F 3 "~" H 2975 1975 50  0001 C CNN
-	1    2975 1975
+P 3025 1975
+F 0 "C10" H 3117 2021 50  0000 L CNN
+F 1 "2.2u" H 3117 1930 50  0000 L CNN
+F 2 "C_0402_1005Metric" H 3025 1975 50  0001 C CNN
+F 3 "~" H 3025 1975 50  0001 C CNN
+	1    3025 1975
 	1    0    0    -1
 $EndComp
@@
 L power:GND #PWR0121
 U 1 1 5DC20B72
-P 2975 2350
-F 0 "#PWR0121" H 2975 2100 50  0001 C CNN
-F 1 "GND" H 2980 2177 50  0000 C CNN
-F 2 "" H 2975 2350 50  0001 C CNN
-F 3 "" H 2975 2350 50  0001 C CNN
-	1    2975 2350
-	1    0    0    -1
-$EndComp
-Wire Wire Line
-	2975 2075 2975 2350
-Wire Wire Line
-	2975 1500 2975 1725
-Wire Wire Line
-	2825 1950 2825 1725
-Wire Wire Line
-	2825 1725 2975 1725
-Connection ~ 2825 1950
-Connection ~ 2975 1725
-Wire Wire Line
-	2975 1725 2975 1875
+P 3025 2350
+F 0 "#PWR0121" H 3025 2100 50  0001 C CNN
+F 1 "GND" H 3030 2177 50  0000 C CNN
+F 2 "" H 3025 2350 50  0001 C CNN
+F 3 "" H 3025 2350 50  0001 C CNN
+	1    3025 2350
+	1    0    0    -1
+$EndComp
+Wire Wire Line
+	3025 2075 3025 2350
+Wire Wire Line
+	3025 1500 3025 1725
+Wire Wire Line
+	2875 1950 2875 1725
+Wire Wire Line
+	2875 1725 3025 1725
+Connection ~ 2875 1950
+Connection ~ 3025 1725
+Wire Wire Line
+	3025 1725 3025 1875
 $Comp
 L power:+3V3 #PWR0122
 U 1 1 5DC2AEA1
-P 2975 1500
-F 0 "#PWR0122" H 2975 1350 50  0001 C CNN
-F 1 "+3V3" H 2990 1673 50  0000 C CNN
-F 2 "" H 2975 1500 50  0001 C CNN
-F 3 "" H 2975 1500 50  0001 C CNN
-	1    2975 1500
+P 3025 1500
+F 0 "#PWR0122" H 3025 1350 50  0001 C CNN
+F 1 "+3V3" H 3040 1673 50  0000 C CNN
+F 2 "" H 3025 1500 50  0001 C CNN
+F 3 "" H 3025 1500 50  0001 C CNN
+	1    3025 1500
 	1    0    0    -1
 $EndComp
@@
 	3200 6650 3200 5825
 Connection ~ 3325 6650
-Text Label 9300 1600 2    50   ~ 0
+Text Label 9300 2100 2    50   ~ 0
 ~SHDN
 Wire Wire Line
-	9300 1600 8925 1600
+	9300 2100 8925 2100
+Wire Wire Line
+	2775 1950 2875 1950
+Wire Wire Line
+	2875 2150 2775 2150
+Wire Wire Line
+	2875 1950 2875 2150
+NoConn ~ 2775 2050
 $EndSCHEMATC
