File: kicad/bias.sch (KiCad schematic (older format))
At the start: 24 parts, among them IC1 LT3571EUD#PBF, IC2 ATSAMD21E18A-AFT, IC3 ADP7118ACPZN3.3, J1 Conn_01x04, J2 CX80B1-24P, J3 Conn_01x03, U1 MCP4726A0T-E_MAY

Commit message: rename
Parts:
- removed C1: 10u, C_0402_1005Metric, symbol Device:C_Small
- added R1, R10, R7: 5.1k, R_0402_1005Metric, symbol Device:R_Small_US
- C2: value 0.1u -> 1u
- J3: footprint footprints:PinHeader_1x03_P2.54mm_Vertical -> footprints:PinHeader_2x02_P2.54mm_Vertical; symbol Connector_Generic:Conn_01x03 -> Connector_Generic:Conn_01x04
Connections:
- net labels added: -5V
- net labels removed: PA02, PA06, PA07
- wire segments 130 -> 132
