File: bias-control/kicad/bias.sch (KiCad schematic (older format))
At the start: 26 parts, among them IC1 LT3571EUD#PBF, IC2 ATSAMD21E18A-AFT, IC3 ADP7118ACPZN3.3, J1 Conn_01x04, J2 CX80B1-24P, J3 Conn_01x03, U1 MCP4726A0T-E_MAY

Commit message: reorg and add tia
Parts:
- C2: value 0.1u -> 1u
Changed lines of the file:
@@
 EESchema Schematic File Version 4
-LIBS:apd-cache
+LIBS:bias-cache
 EELAYER 29 0
 EELAYER END
@@
 P 1425 5000
 F 0 "C2" H 1517 5046 50  0000 L CNN
-F 1 "0.1u" H 1517 4955 50  0000 L CNN
+F 1 "1u" H 1517 4955 50  0000 L CNN
 F 2 "C_0402_1005Metric" H 1425 5000 50  0001 C CNN
 F 3 "" H 1425 5000 50  0001 C CNN
