File: tia/kicad/tia.sch (KiCad schematic (older format))
At the start: 26 parts, among them J1 DF13-5P-1.25DSA, P1 73415-2061, U1 OPA847IDBVT, U2 OPA843IDBVT

Commit message: start routing
Parts:
- removed J1: DF13-5P-1.25DSA, symbol Connector_Generic:Conn_01x05
- added J1: Conn_01x06, footprints:PinHeader_2x03_P2.54mm_Vertical, symbol Connector_Generic:Conn_01x06
Connections:
- net +VDC: now also J1.5 (Pin_5)
- net GND: now also J1.6 (Pin_6)
- net VDDA: now also J1.2 (Pin_2)
- net VSSA: now also J1.3 (Pin_3)
- new net +5V: J1.1 (Pin_1)
- no-connect marks 1 -> 2
Changed lines of the file:
@@
 L power:VDDA #PWR04
 U 1 1 5DBB40A9
-P 1800 1775
-F 0 "#PWR04" H 1800 1625 50  0001 C CNN
-F 1 "VDDA" V 1800 1900 50  0000 L CNN
-F 2 "" H 1800 1775 50  0001 C CNN
-F 3 "" H 1800 1775 50  0001 C CNN
-	1    1800 1775
+P 1250 1425
+F 0 "#PWR04" H 1250 1275 50  0001 C CNN
+F 1 "VDDA" V 1250 1550 50  0000 L CNN
+F 2 "" H 1250 1425 50  0001 C CNN
+F 3 "" H 1250 1425 50  0001 C CNN
+	1    1250 1425
 	0    1    -1   0
 $EndComp
@@
 L power:VSSA #PWR03
 U 1 1 5DBB439F
-P 1800 1675
-F 0 "#PWR03" H 1800 1525 50  0001 C CNN
-F 1 "VSSA" V 1800 1900 50  0000 C CNN
-F 2 "" H 1800 1675 50  0001 C CNN
-F 3 "" H 1800 1675 50  0001 C CNN
-	1    1800 1675
+P 1250 1525
+F 0 "#PWR03" H 1250 1375 50  0001 C CNN
+F 1 "VSSA" V 1250 1750 50  0000 C CNN
+F 2 "" H 1250 1525 50  0001 C CNN
+F 3 "" H 1250 1525 50  0001 C CNN
+	1    1250 1525
 	0    1    -1   0
 $EndComp
-$Comp
-L Connector_Generic:Conn_01x05 J1
-U 1 1 5DBB52A2
-P 1325 1675
-F 0 "J1" H 1405 1717 50  0000 L CNN
-F 1 "DF13-5P-1.25DSA" H 1405 1626 50  0000 L CNN
-F 2 "" H 1325 1675 50  0001 C CNN
-F 3 "" H 1325 1675 50  0001 C CNN
-	1    1325 1675
-	-1   0    0    -1
-$EndComp
-Wire Wire Line
-	1800 1675 1525 1675
-Wire Wire Line
-	1800 1775 1525 1775
-$Comp
-L power:GND #PWR01
-U 1 1 5DBB76FD
-P 1675 2025
-F 0 "#PWR01" H 1675 1775 50  0001 C CNN
-F 1 "GND" H 1680 1852 50  0000 C CNN
-F 2 "" H 1675 2025 50  0001 C CNN
-F 3 "" H 1675 2025 50  0001 C CNN
-	1    1675 2025
-	-1   0    0    -1
-$EndComp
-Wire Wire Line
-	1675 2025 1675 1875
-Wire Wire Line
-	1675 1875 1525 1875
-Wire Wire Line
-	1675 1875 1675 1575
-Wire Wire Line
-	1675 1575 1525 1575
-Connection ~ 1675 1875
+Wire Wire Line
+	1250 1525 975  1525
+Wire Wire Line
+	1250 1425 975  1425
 $Comp
 L power:+VDC #PWR05
 U 1 1 5DBB8157
-P 1850 1325
-F 0 "#PWR05" H 1850 1225 50  0001 C CNN
-F 1 "+VDC" H 1850 1600 50  0000 C CNN
-F 2 "" H 1850 1325 50  0001 C CNN
-F 3 "" H 1850 1325 50  0001 C CNN
-	1    1850 1325
-	-1   0    0    -1
-$EndComp
-Wire Wire Line
-	1850 1325 1850 1475
-Wire Wire Line
-	1850 1475 1525 1475
-Text Label 1775 1475 2    50   ~ 0
+P 1825 1575
+F 0 "#PWR05" H 1825 1475 50  0001 C CNN
+F 1 "+VDC" H 1825 1850 50  0000 C CNN
+F 2 "" H 1825 1575 50  0001 C CNN
+F 3 "" H 1825 1575 50  0001 C CNN
+	1    1825 1575
+	-1   0    0    -1
+$EndComp
+Wire Wire Line
+	1825 1575 1825 1725
+Text Label 1750 1725 2    50   ~ 0
 VBias
 $Comp
@@
 Wire Wire Line
 	10100 4750 10100 5175
+$Comp
+L Connector_Generic:Conn_01x06 J1
+U 1 1 5DBA068E
+P 775 1525
+F 0 "J1" H 693 1942 50  0000 C CNN
+F 1 "Conn_01x06" H 693 1851 50  0000 C CNN
+F 2 "footprints:PinHeader_2x03_P2.54mm_Vertical" H 775 1525 50  0001 C CNN
+F 3 "" H 775 1525 50  0001 C CNN
+	1    775  1525
+	-1   0    0    -1
+$EndComp
+Wire Wire Line
+	1125 1825 975  1825
+Wire Wire Line
+	1125 1975 1125 1825
+$Comp
+L power:GND #PWR01
+U 1 1 5DBB76FD
+P 1125 1975
+F 0 "#PWR01" H 1125 1725 50  0001 C CNN
+F 1 "GND" H 1130 1802 50  0000 C CNN
+F 2 "" H 1125 1975 50  0001 C CNN
+F 3 "" H 1125 1975 50  0001 C CNN
+	1    1125 1975
+	-1   0    0    -1
+$EndComp
+NoConn ~ 975  1625
+Wire Wire Line
+	975  1725 1825 1725
+$Comp
+L power:+5V #PWR0101
+U 1 1 5DBA5394
+P 1150 1000
+F 0 "#PWR0101" H 1150 850 50  0001 C CNN
+F 1 "+5V" H 1165 1173 50  0000 C CNN
+F 2 "" H 1150 1000 50  0001 C CNN
+F 3 "" H 1150 1000 50  0001 C CNN
+	1    1150 1000
+	1    0    0    -1
+$EndComp
+Wire Wire Line
+	975  1325 1150 1325
+Wire Wire Line
+	1150 1325 1150 1000
 $EndSCHEMATC
