File: tia/kicad/tia.sch (KiCad schematic (older format))
At the start: 26 parts, among them J1 Conn_01x06, P1 73415-2061, U1 OPA847IDBVT, U2 OPA843IDBVT

Commit message: choose header
Parts:
- J1: value Conn_01x06 -> SSQ-103-01-G-D
Changed lines of the file:
@@
 Wire Wire Line
 	1250 1425 975  1425
-$Comp
-L power:+VDC #PWR05
-U 1 1 5DBB8157
-P 1825 1575
-F 0 "#PWR05" H 1825 1475 50  0001 C CNN
-F 1 "+VDC" H 1825 1850 50  0000 C CNN
-F 2 "" H 1825 1575 50  0001 C CNN
-F 3 "" H 1825 1575 50  0001 C CNN
-	1    1825 1575
-	-1   0    0    -1
-$EndComp
 Wire Wire Line
 	1825 1575 1825 1725
@@
 P 775 1525
 F 0 "J1" H 693 1942 50  0000 C CNN
-F 1 "Conn_01x06" H 693 1851 50  0000 C CNN
+F 1 "SSQ-103-01-G-D" H 693 1851 50  0000 C CNN
 F 2 "footprints:PinHeader_2x03_P2.54mm_Vertical" H 775 1525 50  0001 C CNN
 F 3 "" H 775 1525 50  0001 C CNN
@@
 Wire Wire Line
 	1150 1325 1150 1000
+$Comp
+L power:+VDC #PWR05
+U 1 1 5DBB8157
+P 1825 1575
+F 0 "#PWR05" H 1825 1475 50  0001 C CNN
+F 1 "+VDC" H 1825 1850 50  0000 C CNN
+F 2 "" H 1825 1575 50  0001 C CNN
+F 3 "" H 1825 1575 50  0001 C CNN
+	1    1825 1575
+	-1   0    0    -1
+$EndComp
 $EndSCHEMATC
