File: tia/kicad/tia.kicad_pcb (KiCad board)
At the start: 2 copper layers, 22 x 22 mm, 25 parts, among them P1 73415-2061, U1 OPA847IDBVT, U2 OPA843IDBVT

Commit message: start routing
Parts:
- added J1: Conn_01x06, footprints:PinHeader_2x03_P2.54mm_Vertical, F.Cu at (206.6, 97.5)
- moved C21 38.8 mm to (197.4, 94.9), turned to 90 degrees
- moved R21 36.0 mm to (197.8, 97.3), turned to 180 degrees
- moved C20 33.0 mm to (191.9, 95.9), turned to 90 degrees
- moved R20 33.0 mm to (191.8, 98.3), turned to 90 degrees
- moved U2 27.5 mm to (194.7, 96.4), turned to -90 degrees
- moved C6 16.1 mm to (208.1, 94.9), turned to 90 degrees
- moved U1 14.2 mm to (180.6, 106.7)
- moved L1 12.2 mm to (184.2, 101.1)
- moved C3 7.33 mm to (204.9, 105.8), turned to -90 degrees
- moved C10 5.56 mm to (204.6, 100.5), turned to -90 degrees
- moved C1 4.94 mm to (203.4, 103.0), turned to -90 degrees
- moved R1 4.45 mm to (195.6, 93.0), turned to 90 degrees
- moved R4 3.76 mm to (206.6, 105.2), turned to -90 degrees
- moved R11 2.39 mm to (204.6, 103.0)
Connections:
- R4 pad 1: (no net) -> +VDC
Routing:
- net VDDA: track 0.00 -> 14.9 mm
- net GND: track 0.00 -> 7.57 mm, vias 0 -> 11
- net VSSA: track 0.00 -> 7.52 mm
- net /OUT: track 0.00 -> 4.69 mm
- net /VBiasFilt: track 0.00 -> 4.26 mm
- net Net-(R23-Pad2): track 0.00 -> 4.05 mm
- net Net-(C3-Pad1): track 0.00 -> 3.50 mm
- net +VDC: track 0.00 -> 2.10 mm

Commit message: choose header
Parts:
- J1: value Conn_01x06 -> SSQ-103-01-G-D
- moved C7 46.3 mm to (198.3, 108.6), turned to -90 degrees
- moved C2 45.6 mm to (195.7, 101.0), turned to 180 degrees
- moved C9 41.8 mm to (196.8, 107.8), turned to 180 degrees
- moved C8 41.1 mm to (199.4, 108.6), turned to -90 degrees
- moved R3 37.8 mm to (200.6, 108.6), turned to 90 degrees
- moved R2 37.0 mm to (195.7, 102.0), turned to 180 degrees
- moved C5 36.4 mm to (195.3, 104.3), turned to 90 degrees
- moved R23 29.8 mm to (194.3, 99.7), turned to 90 degrees
- moved R5 28.6 mm to (192.8, 99.5)
- moved U1 16.9 mm to (197.3, 105.0)
- moved L1 7.09 mm to (190.8, 98.8), turned to 90 degrees
- moved C10 6.60 mm to (208.1, 94.9), turned to 90 degrees
- moved C6 6.58 mm to (204.7, 100.5), turned to -90 degrees
- moved R21 5.44 mm to (192.4, 98.0), turned to 90 degrees
- moved C20 3.29 mm to (194.2, 93.5), turned to 180 degrees
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Connections:
- J1 pad 2: VDDA -> VSSA
- J1 pad 3: VSSA -> VDDA
Routing:
- net VSSA: track 7.52 -> 45.3 mm
- net VDDA: track 14.9 -> 25.4 mm
- net Net-(C2-Pad2): track 0.00 -> 8.75 mm
- net Net-(R1-Pad1): track 0.04 -> 8.20 mm
- net Net-(C2-Pad1): track 0.00 -> 7.57 mm
- net GND: track 7.57 -> 14.0 mm, vias 11 -> 25
- net Net-(C7-Pad1): track 0.00 -> 4.17 mm
- net Net-(R20-Pad1): track 0.00 -> 3.04 mm
- net Net-(L1-Pad1): track 0.00 -> 1.42 mm
- net Net-(R23-Pad2): track 4.05 -> 5.44 mm
- net /OUT: track 4.69 -> 3.88 mm
Other:
- board text added: "SiPM TIA"
- board text removed: "SiPM Bias"
