File: power-supply/kicad/psu.sch (KiCad schematic (older format))
At the start: 13 parts, among them J3 SSQ-103-03-G-D, U1 LM2776, U3 TPS72301DBVR, U5 TPS79333DBVR

Commit message: tweaks, add octopart BOMs
Parts:
- C2: value 10u -> 1u
- C3, C5: value 10u -> 22u
Changed lines of the file:
@@
 P 2350 4825
 F 0 "C2" H 2425 4750 50  0000 C CNN
-F 1 "10u" H 2250 4750 50  0000 C CNN
+F 1 "1u" H 2250 4750 50  0000 C CNN
 F 2 "footprints:C_0603_1608Metric" H 2350 4825 50  0001 L BNN
 F 3 "" H 2350 4825 50  0001 C CNN
@@
 P 4600 4875
 F 0 "C3" H 4675 4800 50  0000 C CNN
-F 1 "10u" H 4500 4800 50  0000 C CNN
+F 1 "22u" H 4500 4800 50  0000 C CNN
 F 2 "footprints:C_0603_1608Metric" H 4600 4875 50  0001 L BNN
 F 3 "" H 4600 4875 50  0001 C CNN
@@
 P 10400 4775
 F 0 "C5" H 10475 4700 50  0000 C CNN
-F 1 "10u" H 10300 4700 50  0000 C CNN
+F 1 "22u" H 10300 4700 50  0000 C CNN
 F 2 "footprints:C_0603_1608Metric" H 10400 4775 50  0001 L BNN
 F 3 "" H 10400 4775 50  0001 C CNN
