File: tiav3_s13360_30XXVE/tiav3_s13360_3030VE.kicad_sch (KiCad schematic)
At the start: 24 parts, among them J1 SSQ-103-01-G-D, J2 Conn_Coaxial, U1 OPA847IDBVT

Commit message: Switch all TIA boards to 0603 for the low pass inductor
0402 is fine for higher cutoffs but its hard to find >1000nH in 0402 without having high resistance.
Parts:
- D2: value s13360_3030VE -> s13360_3050VE
- L2: footprint Inductor_SMD:L_0402_1005Metric -> Inductor_SMD:L_0603_1608Metric
Changed lines of the file:
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@@
 			)
 		)
-		(property "Footprint" "Inductor_SMD:L_0402_1005Metric"
+		(property "Footprint" "Inductor_SMD:L_0603_1608Metric"
 			(at 232.41 110.49 0)
 			(effects
@@
 			)
 		)
-		(property "Value" "s13360_3030VE"
+		(property "Value" "s13360_3050VE"
 			(at 106.68 97.79 90)
 			(effects
