File: tiav3_s14160/kicad/tiav3_s14160.kicad_pcb (KiCad board)
At the start: 4 copper layers, 25.3 x 25.3 mm, 22 parts, among them J1 SSQ-103-01-G-D, J2 Conn_Coaxial, U1 OPA847IDBVT

Commit message: Switch all TIA boards to 0603 for the low pass inductor
0402 is fine for higher cutoffs but its hard to find >1000nH in 0402 without having high resistance.
Parts:
- C8: value 1u -> 22u; footprint Capacitor_SMD:C_0402_1005Metric -> Capacitor_SMD:C_0603_1608Metric
- L2: footprint Inductor_SMD:L_0402_1005Metric -> Inductor_SMD:L_0603_1608Metric
- R2, R23, R3, R5, R7: footprint Resistor_SMD:R_0402_1005Metric_Pad0.72x0.64mm_HandSolder -> Resistor_SMD:R_0402_1005Metric
- moved R7 4.44 mm to (193.6, 97.2), turned to 0 degrees
- moved R3 2.54 mm to (193.6, 98.3), turned to 180 degrees
- moved C8 1.00 mm to (193.6, 99.5), turned to 0 degrees
- moved C3 0.73 mm to (190.5, 101.2)
- moved C7 0.67 mm to (193.6, 100.8), turned to 0 degrees
- moved L2 0.28 mm to (190.4, 103.4)
- moved C2 0.12 mm to (190.4, 105.2)
Routing:
- net GND: track 6.53 -> 8.03 mm
- net Net-(J2-In): track 18.1 -> 17.3 mm
