File: tiav3_s14160/kicad/tiav3_s14160.kicad_sch (KiCad schematic)
At the start: 22 parts, among them J1 SSQ-103-01-G-D, J2 Conn_Coaxial, U1 OPA847IDBVT

Commit message: Switch all TIA boards to 0603 for the low pass inductor
0402 is fine for higher cutoffs but its hard to find >1000nH in 0402 without having high resistance.
Parts:
- C8: value 1u -> 22u; footprint Capacitor_SMD:C_0402_1005Metric -> Capacitor_SMD:C_0603_1608Metric
- L1: footprint footprints:L_0603_1608Metric -> Inductor_SMD:L_0603_1608Metric_Pad1.05x0.95mm_HandSolder
- L2: footprint Inductor_SMD:L_0402_1005Metric -> Inductor_SMD:L_0603_1608Metric
- R1, R2, R23, R3, R5, R7: footprint footprints:R_0402_1005Metric -> Resistor_SMD:R_0402_1005Metric
Changed lines of the file:
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@@
 			)
 		)
-		(property "Footprint" "footprints:R_0402_1005Metric"
+		(property "Footprint" "Resistor_SMD:R_0402_1005Metric"
 			(at 187.96 87.63 0)
 			(effects
@@
 			)
 		)
-		(property "Value" "1u"
+		(property "Value" "22u"
 			(at 172.085 121.285 0)
 			(effects
@@
 			)
 		)
-		(property "Footprint" "Capacitor_SMD:C_0402_1005Metric"
+		(property "Footprint" "Capacitor_SMD:C_0603_1608Metric"
 			(at 171.45 119.38 0)
 			(effects
@@
 			)
 		)
-		(property "Footprint" "footprints:R_0402_1005Metric"
+		(property "Footprint" "Resistor_SMD:R_0402_1005Metric"
 			(at 158.75 119.38 0)
 			(effects
@@
 			)
 		)
-		(property "Footprint" "footprints:L_0603_1608Metric"
+		(property "Footprint" "Inductor_SMD:L_0603_1608Metric_Pad1.05x0.95mm_HandSolder"
 			(at 104.14 120.65 0)
 			(effects
@@
 			)
 		)
-		(property "Footprint" "footprints:R_0402_1005Metric"
+		(property "Footprint" "Resistor_SMD:R_0402_1005Metric"
 			(at 116.84 107.95 0)
 			(effects
@@
 			)
 		)
-		(property "Footprint" "footprints:R_0402_1005Metric"
+		(property "Footprint" "Resistor_SMD:R_0402_1005Metric"
 			(at 104.14 113.03 0)
 			(effects
@@
 			)
 		)
-		(property "Footprint" "footprints:R_0402_1005Metric"
+		(property "Footprint" "Resistor_SMD:R_0402_1005Metric"
 			(at 214.63 110.49 0)
 			(effects
@@
 			)
 		)
-		(property "Footprint" "footprints:R_0402_1005Metric"
+		(property "Footprint" "Resistor_SMD:R_0402_1005Metric"
 			(at 142.24 114.3 0)
 			(effects
@@
 			)
 		)
-		(property "Datasheet" " ~"
+		(property "Datasheet" "~"
 			(at 264.16 110.49 0)
 			(effects
@@
 			)
 		)
-		(property "Footprint" "Inductor_SMD:L_0402_1005Metric"
+		(property "Footprint" "Inductor_SMD:L_0603_1608Metric"
 			(at 232.41 110.49 0)
 			(effects
